File: Main/Main.kicad_pcb (KiCad board)
At the start: 2 copper layers, 147.3 x 70.6 mm, 60 parts, among them J1 Conn_02x03_Odd_Even, J2 Conn_01x06, J3 Conn_01x03, J4 Conn_01x02, J5 Conn_01x12, J6 Conn_01x06, Q1 BCP56, SW1 SW_Push, SW2 SW_Push, SW3 SW_Push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

Commit message: Triac board updated
Parts:
- H1, H2, H3, H4: footprint MountingHole:MountingHole_3.2mm_M3 -> Thermostat:MountingHole_3.2mm_M3
