File: Main/Main.sch (KiCad schematic (older format))
At the start: 60 parts, among them J1 Conn_02x03_Odd_Even, J2 Conn_01x06, J3 Conn_01x03, J4 Conn_01x02, J5 Conn_01x12, J6 Conn_01x06, Q1 BCP56, SW1 SW_Push, SW2 SW_Push, SW3 SW_Push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

Commit message: Triac board updated
Parts:
- H1, H2, H3, H4: footprint MountingHole:MountingHole_3.2mm_M3 -> Thermostat:MountingHole_3.2mm_M3
Changed lines of the file:
@@
 F 0 "H1" H 8500 5646 50  0000 L CNN
 F 1 "MountingHole" H 8500 5555 50  0000 L CNN
-F 2 "MountingHole:MountingHole_3.2mm_M3" H 8400 5600 50  0001 C CNN
+F 2 "Thermostat:MountingHole_3.2mm_M3" H 8400 5600 50  0001 C CNN
 F 3 "~" H 8400 5600 50  0001 C CNN
 	1    8400 5600
@@
 F 0 "H3" H 9200 5646 50  0000 L CNN
 F 1 "MountingHole" H 9200 5555 50  0000 L CNN
-F 2 "MountingHole:MountingHole_3.2mm_M3" H 9100 5600 50  0001 C CNN
+F 2 "Thermostat:MountingHole_3.2mm_M3" H 9100 5600 50  0001 C CNN
 F 3 "~" H 9100 5600 50  0001 C CNN
 	1    9100 5600
@@
 F 0 "H4" H 9900 5646 50  0000 L CNN
 F 1 "MountingHole" H 9900 5555 50  0000 L CNN
-F 2 "MountingHole:MountingHole_3.2mm_M3" H 9800 5600 50  0001 C CNN
+F 2 "Thermostat:MountingHole_3.2mm_M3" H 9800 5600 50  0001 C CNN
 F 3 "~" H 9800 5600 50  0001 C CNN
 	1    9800 5600
@@
 F 0 "H2" H 8500 5896 50  0000 L CNN
 F 1 "MountingHole" H 8500 5805 50  0000 L CNN
-F 2 "MountingHole:MountingHole_3.2mm_M3" H 8400 5850 50  0001 C CNN
+F 2 "Thermostat:MountingHole_3.2mm_M3" H 8400 5850 50  0001 C CNN
 F 3 "~" H 8400 5850 50  0001 C CNN
 	1    8400 5850
