File: Triac/Triac.kicad_pcb (KiCad board)
At the start: 2 copper layers, 147.3 x 70.6 mm, 20 parts, among them J1 Conn_01x06, J2 Conn_01x04, Q1 BT138-600, U1 4N25, U2 MOC3021M

Commit message: Triac board updated
Parts:
- HS1: footprint Thermostat:SK610-94SA -> Thermostat:SK64-37.5
- Q1: footprint Package_TO_SOT_THT:TO-220-3_Vertical -> Package_TO_SOT_THT:TO-220-3_Horizontal_TabDown
- moved R6 58.8 mm to (183.6, 105.2), turned to 270 degrees
- moved C1 40.8 mm to (177.8, 105.2), turned to 90 degrees
- moved J2 30.3 mm to (74.9, 90.2), turned to 270 degrees
- moved C2 27.5 mm to (85.6, 90.2), turned to 270 degrees
- moved R7 21.5 mm to (91.2, 90.2), turned to 270 degrees
- moved HS1 20.3 mm to (133.3, 101.6), turned to 180 degrees
- moved Q1 5.92 mm to (135.9, 79.2)
- moved R5 1.08 mm to (193.5, 105.9), turned to 0 degrees
Connections:
- J2 pad 1: /AC_OUT -> /AC_L
- J2 pad 4: /AC_L -> /AC_OUT
Routing:
- net Net-(C1-Pad1): track 69.4 -> 15.3 mm, vias 1 -> 0
- net /AC_OUT: track 0.00 -> 46.7 mm
- net /AC_N: track 130.3 -> 119.9 mm, vias 0 -> 2
- net Net-(Q1-Pad3): track 86.5 -> 78.4 mm, vias 0 -> 1
- net /AC_L: track 81.5 -> 76.3 mm, vias 1 -> 0
- net Net-(C2-Pad1): track 4.44 -> 5.97 mm
- added copper zone on F.Cu, net /AC_L
- added copper zone on F.Cu, net /AC_N
- removed copper zone on B.Cu, net /AC_L
- removed copper zone on B.Cu, net /AC_N
Other:
- board size 147.3 x 70.6 mm -> 147.3 x 46 mm
- net class AC: trace_width 0.5 -> 1

Commit message: Triac board updated
Parts:
- H1, H2, H3, H4: footprint MountingHole:MountingHole_3.2mm_M3 -> Thermostat:MountingHole_3.2mm_M3
Routing:
- net /AC_L: track 76.3 -> 85.1 mm
- net /AC_N: track 119.9 -> 126.6 mm
