File: Triac/Triac.sch (KiCad schematic (older format))
At the start: 20 parts, among them J1 Conn_01x06, J2 Conn_01x04, Q1 BT138-600, U1 4N25, U2 MOC3021M

Commit message: Triac board updated
Parts:
- HS1: footprint Thermostat:SK610-94SA -> Thermostat:SK64-37.5
- Q1: footprint Package_TO_SOT_THT:TO-220-3_Vertical -> Package_TO_SOT_THT:TO-220-3_Horizontal_TabDown
Connections:
- net AC_L: now also J2.1 (Pin_1); no longer J2.4 (Pin_4)
- net AC_OUT: now also J2.4 (Pin_4); no longer J2.1 (Pin_1)
Changed lines of the file:
@@
 F 0 "Q1" H 5978 2246 50  0000 L CNN
 F 1 "BT138-600" H 5978 2155 50  0000 L CNN
-F 2 "Package_TO_SOT_THT:TO-220-3_Vertical" H 6050 2125 50  0001 L CIN
+F 2 "Package_TO_SOT_THT:TO-220-3_Horizontal_TabDown" H 6050 2125 50  0001 L CIN
 F 3 "https://assets.nexperia.com/documents/data-sheet/BT138_SER_D_E.pdf" H 5850 2200 50  0001 L CNN
 	1    5850 2200
@@
 Connection ~ 4950 4250
 Connection ~ 4950 4550
-Text Label 9000 3050 2    50   ~ 0
+Text Label 9000 3350 2    50   ~ 0
 AC_OUT
 Text Label 9000 3150 2    50   ~ 0
 AC_N
-Text Label 9000 3350 2    50   ~ 0
+Text Label 9000 3050 2    50   ~ 0
 AC_L
 $Comp
@@
 F 0 "HS1" H 9942 5021 50  0000 L CNN
 F 1 "Heatsink" H 9942 4930 50  0000 L CNN
-F 2 "Thermostat:SK610-94SA" H 9812 4900 50  0001 C CNN
+F 2 "Thermostat:SK64-37.5" H 9812 4900 50  0001 C CNN
 F 3 "~" H 9812 4900 50  0001 C CNN
 	1    9800 4900

Commit message: Triac board updated
Parts:
- H1, H2, H3, H4: footprint MountingHole:MountingHole_3.2mm_M3 -> Thermostat:MountingHole_3.2mm_M3
Changed lines of the file:
@@
 F 0 "H1" H 8500 5646 50  0000 L CNN
 F 1 "MountingHole" H 8500 5555 50  0000 L CNN
-F 2 "MountingHole:MountingHole_3.2mm_M3" H 8400 5600 50  0001 C CNN
+F 2 "Thermostat:MountingHole_3.2mm_M3" H 8400 5600 50  0001 C CNN
 F 3 "~" H 8400 5600 50  0001 C CNN
 	1    8400 5600
@@
 F 0 "H3" H 9200 5646 50  0000 L CNN
 F 1 "MountingHole" H 9200 5555 50  0000 L CNN
-F 2 "MountingHole:MountingHole_3.2mm_M3" H 9100 5600 50  0001 C CNN
+F 2 "Thermostat:MountingHole_3.2mm_M3" H 9100 5600 50  0001 C CNN
 F 3 "~" H 9100 5600 50  0001 C CNN
 	1    9100 5600
@@
 F 0 "H4" H 9900 5646 50  0000 L CNN
 F 1 "MountingHole" H 9900 5555 50  0000 L CNN
-F 2 "MountingHole:MountingHole_3.2mm_M3" H 9800 5600 50  0001 C CNN
+F 2 "Thermostat:MountingHole_3.2mm_M3" H 9800 5600 50  0001 C CNN
 F 3 "~" H 9800 5600 50  0001 C CNN
 	1    9800 5600
@@
 F 0 "H2" H 8500 5896 50  0000 L CNN
 F 1 "MountingHole" H 8500 5805 50  0000 L CNN
-F 2 "MountingHole:MountingHole_3.2mm_M3" H 8400 5850 50  0001 C CNN
+F 2 "Thermostat:MountingHole_3.2mm_M3" H 8400 5850 50  0001 C CNN
 F 3 "~" H 8400 5850 50  0001 C CNN
 	1    8400 5850
